File: dmem_2V0.kicad_pcb (KiCad board)
At the start: 4 copper layers, 189 x 72 mm, 166 parts, among them J1 D15P33E4GV00LF, J10 7701-3, J11 7701-3, J2 T1M-03-F-SV-L, J3 T1M-03-F-SV-L, J4 T1M-03-F-SV-L, J5 T1M-03-F-SV-L, J6 T1M-03-F-SV-L, J7 T1M-03-F-SV-L, J8 T1M-03-F-SV-L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

Commit message: Changed R25,R24,R59,R58 values from 1K5 to 1K2.
Parts:
- R24, R25, R58, R59: value 1K5 -> 1K2
Changed lines of the file:
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@@
         (effects (font (size 1 1) (thickness 0.15)))
     )
-    (fp_text value "1K5" (at 0 1.65 90) (layer "F.Fab") hide
+    (fp_text value "1K2" (at 0 1.65 90) (layer "F.Fab") hide
         (effects (font (size 1 1) (thickness 0.15)))
     )
@@
         (effects (font (size 1 1) (thickness 0.15)))
     )
-    (fp_text value "1K5" (at 0 1.65 90) (layer "F.Fab") hide
+    (fp_text value "1K2" (at 0 1.65 90) (layer "F.Fab") hide
         (effects (font (size 1 1) (thickness 0.15)))
     )
@@
         (effects (font (size 1 1) (thickness 0.15)))
     )
-    (fp_text value "1K5" (at 0 1.65 90) (layer "F.Fab") hide
+    (fp_text value "1K2" (at 0 1.65 90) (layer "F.Fab") hide
         (effects (font (size 1 1) (thickness 0.15)))
     )
@@
         (effects (font (size 1 1) (thickness 0.15)))
     )
-    (fp_text value "1K5" (at 0 1.65 90) (layer "F.Fab") hide
+    (fp_text value "1K2" (at 0 1.65 90) (layer "F.Fab") hide
         (effects (font (size 1 1) (thickness 0.15)))
     )

Commit message: Removed R30, R31 and mirrors
Parts:
- removed R30, R31, R60, R61: 1K5, Resistor_SMD:R_0805_2012Metric
Routing:
- net /cold_amplifier_ch2/output-: track 45.4 -> 38.0 mm, vias 3 -> 2
- net /cold_amplifier_ch1/output-: track 45.4 -> 38.0 mm, vias 3 -> 2
- net /cold_amplifier_ch2/output+: track 45.3 -> 38.1 mm, vias 3 -> 2
- net /cold_amplifier_ch1/output+: track 45.3 -> 38.1 mm, vias 3 -> 2
