File: cold_amplifier_ch1.kicad_sch (KiCad schematic)
At the start: 30 parts, among them J2 T1M-03-F-SV-L, J3 T1M-03-F-SV-L, J4 T1M-03-F-SV-L, J5 T1M-03-F-SV-L

Commit message: Changed R25,R24,R59,R58 values from 1K5 to 1K2.
Parts:
- R1: value 1K5 -> 1K2
Changed lines of the file:
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@@
       (effects (font (size 1.27 1.27)))
     )
-    (property "Value" "1K5" (at 144.78 123.19 90)
+    (property "Value" "1K2" (at 144.78 123.19 90)
       (effects (font (size 1.27 1.27)))
     )
@@
       (effects (font (size 1.27 1.27)))
     )
-    (property "Value" "1K5" (at 143.51 55.88 90)
+    (property "Value" "1K2" (at 143.51 55.88 90)
       (effects (font (size 1.27 1.27)))
     )

Commit message: Removed R30, R31 and mirrors
Parts:
- removed R1 (x2): 1K5, Resistor_SMD:R_0805_2012Metric, symbol Device:R_US
Changed lines of the file:
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@@
   (junction (at 74.93 104.14) (diameter 0) (color 0 0 0 0)
   )
-  (junction (at 189.23 91.44) (diameter 0) (color 0 0 0 0)
-  )
   (junction (at 17.78 163.83) (diameter 0) (color 0 0 0 0)
   )
@@
   (junction (at 17.78 102.87) (diameter 0) (color 0 0 0 0)
   )
-  (junction (at 189.23 104.14) (diameter 0) (color 0 0 0 0)
-  )
   (junction (at 17.78 73.66) (diameter 0) (color 0 0 0 0)
   )
@@
     (stroke (width 0) (type default))
   )
-  (wire (pts (xy 189.23 80.01) (xy 189.23 91.44))
-    (stroke (width 0) (type default))
-  )
   (wire (pts (xy 17.78 135.89) (xy 17.78 163.83))
     (stroke (width 0) (type default))
@@
     (stroke (width 0) (type default))
   )
-  (wire (pts (xy 189.23 104.14) (xy 189.23 114.3))
-    (stroke (width 0) (type default))
-  )
   (wire (pts (xy 52.07 162.56) (xy 57.15 162.56))
     (stroke (width 0) (type default))
@@
     (stroke (width 0) (type default))
   )
-  (wire (pts (xy 189.23 121.92) (xy 189.23 127))
-    (stroke (width 0) (type default))
-  )
-  (wire (pts (xy 189.23 64.77) (xy 189.23 72.39))
-    (stroke (width 0) (type default))
-  )
   (wire (pts (xy 88.9 104.14) (xy 74.93 104.14))
     (stroke (width 0) (type default))
@@
     (stroke (width 0) (type default))
   )
-  (wire (pts (xy 189.23 91.44) (xy 194.31 91.44))
+  (wire (pts (xy 184.15 91.44) (xy 194.31 91.44))
     (stroke (width 0) (type default))
   )
@@
     (stroke (width 0) (type default))
   )
-  (wire (pts (xy 189.23 104.14) (xy 194.31 104.14))
+  (wire (pts (xy 184.15 104.14) (xy 194.31 104.14))
     (stroke (width 0) (type default))
   )
@@
     (stroke (width 0) (type default))
   )
-  (wire (pts (xy 184.15 104.14) (xy 189.23 104.14))
-    (stroke (width 0) (type default))
-  )
   (wire (pts (xy 113.03 73.66) (xy 113.03 76.2))
     (stroke (width 0) (type default))
@@
   )
   (wire (pts (xy 48.26 135.89) (xy 44.45 135.89))
-    (stroke (width 0) (type default))
-  )
-  (wire (pts (xy 184.15 91.44) (xy 189.23 91.44))
     (stroke (width 0) (type default))
   )
@@
         (path "/3e9c66f9-4dd4-413a-a9f0-4be475bcdd89/1456cace-ae68-405a-8445-6ed61c30fb1f"
           (reference "C32") (unit 1)
-        )
-      )
-    )
-  )
-  (symbol (lib_id "Device:R_US") (at 189.23 76.2 0) (unit 1)
-    (in_bom yes) (on_board yes) (dnp no) (fields_autoplaced)
-    (property "Reference" "R1" (at 191.77 74.93 0)
-      (effects (font (size 1.27 1.27)) (justify left))
-    )
-    (property "Value" "1K5" (at 191.77 77.47 0)
-      (effects (font (size 1.27 1.27)) (justify left))
-    )
-    (property "Footprint" "Resistor_SMD:R_0805_2012Metric" (at 190.246 76.454 90)
-      (effects (font (size 1.27 1.27)) hide)
-    )
-    (property "Datasheet" "~" (at 189.23 76.2 0)
-      (effects (font (size 1.27 1.27)) hide)
-    )
-    (pin "1")
-    (pin "2")
-    (instances
-      (project "dmem_2V0"
-        (path "/3e9c66f9-4dd4-413a-a9f0-4be475bcdd89/3c1290f2-1529-4d1d-8df3-34847770d53c/4ff7a2e6-97e8-4e4f-9ffd-036809f49006"
-          (reference "R1") (unit 1)
-        )
-        (path "/3e9c66f9-4dd4-413a-a9f0-4be475bcdd89/3c1290f2-1529-4d1d-8df3-34847770d53c"
-          (reference "R30") (unit 1)
-        )
-        (path "/3e9c66f9-4dd4-413a-a9f0-4be475bcdd89/1456cace-ae68-405a-8445-6ed61c30fb1f"
-          (reference "R60") (unit 1)
         )
       )
@@
     )
   )
-  (symbol (lib_id "power:GND") (at 189.23 127 0) (unit 1)
-    (in_bom yes) (on_board yes) (dnp no) (fields_autoplaced)
-    (property "Reference" "#PWR017" (at 189.23 133.35 0)
-      (effects (font (size 1.27 1.27)) hide)
-    )
-    (property "Value" "GND" (at 189.23 132.08 0)
-      (effects (font (size 1.27 1.27)))
-    )
-    (property "Footprint" "" (at 189.23 127 0)
-      (effects (font (size 1.27 1.27)) hide)
-    )
-    (property "Datasheet" "" (at 189.23 127 0)
-      (effects (font (size 1.27 1.27)) hide)
-    )
-    (pin "1")
-    (instances
-      (project "dmem_2V0"
-        (path "/3e9c66f9-4dd4-413a-a9f0-4be475bcdd89/3c1290f2-1529-4d1d-8df3-34847770d53c"
-          (reference "#PWR017") (unit 1)
-        )
-        (path "/3e9c66f9-4dd4-413a-a9f0-4be475bcdd89/1456cace-ae68-405a-8445-6ed61c30fb1f"
-          (reference "#PWR034") (unit 1)
-        )
-      )
-    )
-  )
   (symbol (lib_id "Device:C") (at 113.03 91.44 90) (unit 1)
     (in_bom yes) (on_board yes) (dnp no) (fields_autoplaced)
@@
     )
   )
-  (symbol (lib_id "Device:R_US") (at 189.23 118.11 0) (unit 1)
-    (in_bom yes) (on_board yes) (dnp no) (fields_autoplaced)
-    (property "Reference" "R1" (at 191.77 116.84 0)
-      (effects (font (size 1.27 1.27)) (justify left))
-    )
-    (property "Value" "1K5" (at 191.77 119.38 0)
-      (effects (font (size 1.27 1.27)) (justify left))
-    )
-    (property "Footprint" "Resistor_SMD:R_0805_2012Metric" (at 190.246 118.364 90)
-      (effects (font (size 1.27 1.27)) hide)
-    )
-    (property "Datasheet" "~" (at 189.23 118.11 0)
-      (effects (font (size 1.27 1.27)) hide)
-    )
-    (pin "1")
-    (pin "2")
-    (instances
-      (project "dmem_2V0"
-        (path "/3e9c66f9-4dd4-413a-a9f0-4be475bcdd89/3c1290f2-1529-4d1d-8df3-34847770d53c/4ff7a2e6-97e8-4e4f-9ffd-036809f49006"
-          (reference "R1") (unit 1)
-        )
-        (path "/3e9c66f9-4dd4-413a-a9f0-4be475bcdd89/3c1290f2-1529-4d1d-8df3-34847770d53c"
-          (reference "R31") (unit 1)
-        )
-        (path "/3e9c66f9-4dd4-413a-a9f0-4be475bcdd89/1456cace-ae68-405a-8445-6ed61c30fb1f"
-          (reference "R61") (unit 1)
-        )
-      )
-    )
-  )
   (symbol (lib_id "Device:R_US") (at 60.96 162.56 270) (mirror x) (unit 1)
     (in_bom yes) (on_board yes) (dnp no)
@@
         )
       )
-    )
-  )
-  (symbol (lib_id "power:GND") (at 189.23 64.77 180) (unit 1)
-    (in_bom yes) (on_board yes) (dnp no) (fields_autoplaced)
-    (property "Reference" "#PWR018" (at 189.23 58.42 0)
-      (effects (font (size 1.27 1.27)) hide)
-    )
-    (property "Value" "GND" (at 189.23 59.69 0)
-      (effects (font (size 1.27 1.27)))
-    )
-    (property "Footprint" "" (at 189.23 64.77 0)
-      (effects (font (size 1.27 1.27)) hide)
-    )
-    (property "Datasheet" "" (at 189.23 64.77 0)
-      (effects (font (size 1.27 1.27)) hide)
-    )
-    (pin "1")
-    (instances
-      (project "dmem_2V0"
-        (path "/3e9c66f9-4dd4-413a-a9f0-4be475bcdd89/3c1290f2-1529-4d1d-8df3-34847770d53c"
-          (reference "#PWR018") (unit 1)
-        )
-        (path "/3e9c66f9-4dd4-413a-a9f0-4be475bcdd89/1456cace-ae68-405a-8445-6ed61c30fb1f"
-          (reference "#PWR033") (unit 1)
-        )
-      )

Commit message: Moved connectors SiPM flex connectorsto both sides; rectangular vias stitching pattern
Parts:
- C5: Digikey Part Number (none) -> 490-GRM3195C2A104JA01DCT-ND; Manufacturer (none) -> Murata Electronics; Part Number (none) -> GRM3195C2A104JA01D
- J2: Digikey Part (none) -> SAM15301CT-ND; Manufacturer Name (none) -> SAMTEC; Part Number (none) -> T1M-03-F-SV-L
- J3, J4, J5: Description  (none) -> Connector Header Surface Mount 3 position 0.039" (1.00mm); Digikey Part Number (none) -> SAM15301CT-ND; Manufacturer Name (none) -> SAMTEC; Part Number (none) -> T1M-03-F-SV-L
- R1: Digikey Part Number (none) -> 749-MCU0805MZ0000ZP500CT-ND; Manufacturer (none) -> Vishay Beyschlag/Draloric/BC Components; Part Number (none) -> MCU0805MZ0000ZP500
- R1: Digikey Part Number (none) -> P1.2KDACT-ND; Manufacturer (none) -> Panasonic Electronic Components; Part Number (none) -> ERA-6AEB122V
- R1: Digikey Part Number (none) -> 13-RT0805BRD071RLCT-ND; Manufacturer (none) -> YAGEO; Part Number (none) -> RT0805BRD071RL
- R1: Digikey Part Number (none) -> P49.9DACT-ND; Manufacturer (none) -> Panasonic Electronic Components; Part Number (none) -> ERA-6AEB49R9V
